Commit message: Update meshes

File: motoman_gp12_support/urdf/gp12_macro.xacro (robot description, xacro)
@@ -156,5 +156,4 @@
     </joint>
     <!-- ROS-Industrial 'tool0' frame: all-zeros tool frame -->
-    <link name="${prefix}tool0" />
     <joint name="${prefix}flange-tool0" type="fixed">
         <origin xyz="0 0 0" rpy="${radians(180)} ${radians(-90)} 0" />
